Commit message: add gpio interface

File: src/water_bot_control/description/ros2_control/diffbot.ros2_control.xacro (robot description, xacro)
@@ -12,5 +12,5 @@
       <hardware>
         <plugin>water_bot_control/WarterBotHardware</plugin>
-        <param name = "wheel_radius">20.00</param>
+        <param name = "wheel_radius">100.00</param>
       </hardware>
       <xacro:if value="${use_mock_hardware}">
@@ -30,4 +30,9 @@
         <state_interface name="velocity"/>
       </joint>
+      <gpio name = "${prefix}water_bot_IOs">
+        <command_interface name="clean_mode"/>
+        <state_interface name="op_mode"/>
+        <state_interface name="clean_mode"/>
+      </gpio>
     </ros2_control>
   </xacro:macro>

File: src/water_bot_description/diffbot/urdf/diffbot_description.urdf.xacro (robot description, xacro)
@@ -125,5 +125,5 @@
           <sphere radius="${caster_wheel_radius}"/>
         </geometry>
-        <material name="white"/>
+        <material name="red"/>
       </visual>
       <inertial>
@@ -168,5 +168,5 @@
       <parent link="${prefix}base_link"/>
       <child link="${prefix}lidar_link"/>
-      <origin xyz="0 0 ${base_height/2 + lidar_height/2}" rpy="0 0 0"/>
+      <origin xyz="0 0 ${base_height/2 + lidar_height/2}" rpy="0 0 ${PI}"/>
     </joint>
     <!-- lidar Link -->
